File: dev_board/Dev_board_V0.3/Nrf52480_Dev_board/nRF52840.kicad_sch (KiCad schematic)
At the start: 17 parts, among them J1 Conn_01x05, J10 Conn_01x02, J11 Conn_01x05, J3 SWD Debug connector, J6 Conn_01x07, J7 Conn_01x02, SW5 SW_Push, U1 MDBT50Q-1MV2, Y1 32.768KHz

Commit message: updated BOM
Parts:
- J1, J10, J11, J6, J7: now left out of the parts list
Changed lines of the file:
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@@
 		(unit 1)
 		(exclude_from_sim no)
-		(in_bom yes)
+		(in_bom no)
 		(on_board yes)
 		(dnp no)
@@
 		(unit 1)
 		(exclude_from_sim no)
-		(in_bom yes)
+		(in_bom no)
 		(on_board yes)
 		(dnp no)
@@
 		(unit 1)
 		(exclude_from_sim no)
-		(in_bom yes)
+		(in_bom no)
 		(on_board yes)
 		(dnp no)
@@
 		(unit 1)
 		(exclude_from_sim no)
-		(in_bom yes)
+		(in_bom no)
 		(on_board yes)
 		(dnp no)
@@
 		(unit 1)
 		(exclude_from_sim no)
-		(in_bom yes)
-		(on_board yes)
-		(dnp no)
+		(in_bom no)
+		(on_board yes)
+		(dnp no)
